File: led spot/led spot.sch (KiCad schematic (older format))
At the start: 22 parts, among them P1 LUX, P2 LED, P3 SWD, U1 MAX15062, U2 STM32F030-20, U3 ISL83485IBZ, U4 2CH-TVS

Commit message: Better schematic @ervanalb
Parts:
- removed D3: 3V3, ~, symbol LED
- removed R5: 680, ~, symbol R
- added C8: 1uF, ~, symbol C
Connections:
- net +48V: now also C8.1
- net GND: now also R1.1, C8.2; no longer R3.2
- net PWM_G: now also U2.12 (PA6); no longer U2.9 (PA3)
- net PWM_R: now also U2.13 (PA7); no longer U2.8 (PA2)
- net UART_DIR: now also U2.14 (PB1); no longer U2.12 (PA6)
- net VCC: now also R3.2; no longer R1.1
Other:
- note added: "TIM3_CH1"
- note added: "TIM3_CH2"
- note removed: "TIM15_CH1"
- note removed: "TIM15_CH2"
- moved on the sheet: D2, D4, R4, R6
