File: led spot/led_driver.sch (KiCad schematic (older format))
At the start: 6 parts, among them U5 TPS92511

Commit message: Better schematic @ervanalb
Parts:
- added C9: 1uF, ~, symbol C
Connections:
- net GND: now also C9.2
- net Vin: now also C9.1
Changed lines of the file:
@@
 $Descr A4 11693 8268
 encoding utf-8
-Sheet 2 4
+Sheet 4 4
 Title ""
-Date "2 jun 2015"
+Date "4 jun 2015"
 Rev ""
 Comp ""
@@
 P 6050 4150
 AR Path="/556D27B1/556D2B65" Ref="#PWR030"  Part="1"
-AR Path="/556D3024/556D2B65" Ref="#PWR035"  Part="1"
-AR Path="/556D375F/556D2B65" Ref="#PWR040"  Part="1"
-F 0 "#PWR040" H 6050 4150 30  0001 C CNN
+AR Path="/556D3024/556D2B65" Ref="#PWR036"  Part="1"
+AR Path="/556D375F/556D2B65" Ref="#PWR042"  Part="1"
+F 0 "#PWR042" H 6050 4150 30  0001 C CNN
 F 1 "GND" H 6050 4080 30  0001 C CNN
 F 2 "" H 6050 4150 60  0000 C CNN
@@
 P 4250 4150
 AR Path="/556D27B1/556D2BA7" Ref="#PWR031"  Part="1"
-AR Path="/556D3024/556D2BA7" Ref="#PWR036"  Part="1"
-AR Path="/556D375F/556D2BA7" Ref="#PWR041"  Part="1"
-F 0 "#PWR041" H 4250 4150 30  0001 C CNN
+AR Path="/556D3024/556D2BA7" Ref="#PWR037"  Part="1"
+AR Path="/556D375F/556D2BA7" Ref="#PWR043"  Part="1"
+F 0 "#PWR043" H 4250 4150 30  0001 C CNN
 F 1 "GND" H 4250 4080 30  0001 C CNN
 F 2 "" H 4250 4150 60  0000 C CNN
@@
 P 4100 4150
 AR Path="/556D27B1/556D2BD6" Ref="#PWR032"  Part="1"
-AR Path="/556D3024/556D2BD6" Ref="#PWR037"  Part="1"
-AR Path="/556D375F/556D2BD6" Ref="#PWR042"  Part="1"
-F 0 "#PWR042" H 4100 4150 30  0001 C CNN
+AR Path="/556D3024/556D2BD6" Ref="#PWR038"  Part="1"
+AR Path="/556D375F/556D2BD6" Ref="#PWR044"  Part="1"
+F 0 "#PWR044" H 4100 4150 30  0001 C CNN
 F 1 "GND" H 4100 4080 30  0001 C CNN
 F 2 "" H 4100 4150 60  0000 C CNN
@@
 P 3950 4150
 AR Path="/556D27B1/556D2BEF" Ref="#PWR033"  Part="1"
-AR Path="/556D3024/556D2BEF" Ref="#PWR038"  Part="1"
-AR Path="/556D375F/556D2BEF" Ref="#PWR043"  Part="1"
-F 0 "#PWR043" H 3950 4150 30  0001 C CNN
+AR Path="/556D3024/556D2BEF" Ref="#PWR039"  Part="1"
+AR Path="/556D375F/556D2BEF" Ref="#PWR045"  Part="1"
+F 0 "#PWR045" H 3950 4150 30  0001 C CNN
 F 1 "GND" H 3950 4080 30  0001 C CNN
 F 2 "" H 3950 4150 60  0000 C CNN
@@
 P 3800 4150
 AR Path="/556D27B1/556D2C35" Ref="#PWR034"  Part="1"
-AR Path="/556D3024/556D2C35" Ref="#PWR039"  Part="1"
-AR Path="/556D375F/556D2C35" Ref="#PWR044"  Part="1"
-F 0 "#PWR044" H 3800 4150 30  0001 C CNN
+AR Path="/556D3024/556D2C35" Ref="#PWR040"  Part="1"
+AR Path="/556D375F/556D2C35" Ref="#PWR046"  Part="1"
+F 0 "#PWR046" H 3800 4150 30  0001 C CNN
 F 1 "GND" H 3800 4080 30  0001 C CNN
 F 2 "" H 3800 4150 60  0000 C CNN
@@
 Wire Wire Line
 	3800 4150 3800 4000
+Text HLabel 3300 3500 0    60   Input ~ 0
+Vin
+$Comp
+L C C9
+U 1 1 556FFD7B
+P 3550 3800
+AR Path="/556D27B1/556FFD7B" Ref="C9"  Part="1"
+AR Path="/556D375F/556FFD7B" Ref="C11"  Part="1"
+AR Path="/556D3024/556FFD7B" Ref="C10"  Part="1"
+F 0 "C11" H 3550 3900 40  0000 L CNN
+F 1 "1uF" H 3556 3715 40  0000 L CNN
+F 2 "~" H 3588 3650 30  0000 C CNN
+F 3 "~" H 3550 3800 60  0000 C CNN
+	1    3550 3800
+	1    0    0    -1
+$EndComp
+Wire Wire Line
+	3300 3500 3550 3500
+Wire Wire Line
+	3550 3500 3550 3600
+$Comp
+L GND #PWR035
+U 1 1 556FFDA1
+P 3550 4150
+AR Path="/556D27B1/556FFDA1" Ref="#PWR035"  Part="1"
+AR Path="/556D375F/556FFDA1" Ref="#PWR047"  Part="1"
+AR Path="/556D3024/556FFDA1" Ref="#PWR041"  Part="1"
+F 0 "#PWR047" H 3550 4150 30  0001 C CNN
+F 1 "GND" H 3550 4080 30  0001 C CNN
+F 2 "" H 3550 4150 60  0000 C CNN
+F 3 "" H 3550 4150 60  0000 C CNN
+	1    3550 4150
+	1    0    0    -1
+$EndComp
+Wire Wire Line
+	3550 4150 3550 4000
 $EndSCHEMATC
