File: led_strip_hardware/unified.kicad_pcb (KiCad board)
At the start: 4 copper layers, 48.3 x 20.3 mm, 36 parts, among them P1 mod_jack_in, P2 PWR_TST, P3 LED_STRIP, P4 ICSP, Q1 FDN5618P, SW1 USR_SW, U1 ISL83485IBZ, U2 TPS54560, U3 STM32F030-32, U4 NCP1117ST33T3G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

Commit message: Progress on v7 of led_strip_hardware
Parts:
- R5: value 68K -> 270K
- R6: value 12K -> 22K
Routing:
- added copper zone on F.Cu, net GND

Commit message: Progress on v7 of led_strip_hardware; some lux utilities
Parts:
- added C10: 2u2, SM1210, F.Cu at (127.8, 110.7)
- added C11: 2u2, SA0805, B.Cu at (130.8, 109.5)
- added C12: 100n, SA0402, B.Cu at (144.8, 122.2)
- Q1, R10, R9: moved to B.Cu
- moved R10 17.1 mm to (117.3, 122.2)
- moved R9 15.1 mm to (118.9, 122.2)
- moved Q1 12.2 mm to (121.7, 122.2)
- moved C2 2.69 mm to (130.8, 113.3), turned to 0 degrees
- moved C9 1.73 mm to (130.8, 111.5), turned to 180 degrees
Routing:
- net Net-(D3-Pad2): track 24.9 -> 11.1 mm, vias 1 -> 0
- net 3V3: track 62.3 -> 67.1 mm
- net /DAT: track 16.2 -> 19.2 mm
- net +48V: track 27.7 -> 29.5 mm
- net Net-(Q1-PadG): track 3.41 -> 3.92 mm
Other:
- board text added: "Digital LED Strip rev 7"
- board text added: "Eric Van Albert Zach Banks"
- board text added: "github.com/ervanalb/lux"
- board text removed: "Digital LED Strip Driver"
- board text removed: "Eric Van Albert"
- board text removed: "rev 6"

Commit message: LED hardware rev 7
Parts:
- moved U4 14.9 mm to (144.8, 122.9), turned to 270 degrees
- moved L1 14.4 mm to (136.7, 122.9), turned to 270 degrees
- moved D2 7.76 mm to (133.1, 112.8)
- moved C3 3.66 mm to (129.0, 117.1)
- moved C11 3.33 mm to (134.0, 110.5), turned to 270 degrees
- moved R4 2.79 mm to (136.4, 121.3), turned to 0 degrees
- moved D1 2.29 mm to (130.8, 122.9)
- moved R5 2.07 mm to (127.0, 125.0)
- moved R6 1.98 mm to (128.3, 125.0)
- moved U2 1.70 mm to (129.0, 120.7)
- moved C5 1.61 mm to (132.1, 125.0)
- moved C4 1.57 mm to (130.8, 125.0)
- moved R3 1.55 mm to (129.5, 125.0)
- moved R2 1.53 mm to (125.7, 125.0)
- moved C9 1.44 mm to (131.8, 110.5), turned to 270 degrees
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Connections:
- U3 pad 27: Net-(U3-Pad27) -> Net-(SW1-Pad3)
- U3 pad 30: Net-(SW1-Pad3) -> Net-(U3-Pad30)
Routing:
- net GND: track 139.9 -> 115.0 mm, vias 54 -> 50
- net Net-(C3-Pad2): track 0.44 -> 24.3 mm
- net 3V3: track 67.1 -> 78.3 mm
- net Net-(R4-Pad2): track 5.68 -> 2.04 mm
- net Net-(D1-Pad1): track 2.06 -> 5.25 mm
- net /DAT: track 19.2 -> 16.2 mm
- net VPP: track 44.6 -> 47.6 mm
- net Net-(C3-Pad1): track 5.72 -> 3.79 mm
- net Net-(SW1-Pad3): track 5.51 -> 4.51 mm
- net Net-(R5-Pad2): track 7.98 -> 7.17 mm
- net Net-(C5-Pad1): track 7.48 -> 8.28 mm
- removed copper zone on F.Cu, net Net-(C3-Pad2)
