File: led_spot_hardware/led_driver.sch (KiCad schematic (older format))
At the start: 7 parts, among them U5 TPS92511

Commit message: improvements to LED spot
Parts:
- added R13: 1K, Resistors_SMD:R_0603, symbol R
- C10: footprint (none) -> Capacitors_SMD:C_0805; symbol C -> C-RESCUE-led_spot
- C5: footprint ~ -> Capacitors_SMD:C_0603; symbol C -> C-RESCUE-led_spot
- D5: footprint ~ -> Diodes_SMD:SMB_Standard
- L2: footprint ~ -> custom:NRS6028T101MMGJ
- R7, R8: footprint ~ -> Resistors_SMD:R_0603; symbol R -> R-RESCUE-led_spot
- U5: footprint (none) -> Housings_SOIC:SOIC-8-1EP_3.9x4.9mm_Pitch1.27mm
Connections:
- wire segments 20 -> 22
Changed lines of the file:
@@
 EESchema Schematic File Version 2
+LIBS:led spot-rescue
 LIBS:power
 LIBS:device
@@
 LIBS:max15062
 LIBS:custom
+LIBS:switches
 LIBS:led spot-cache
-EELAYER 24 0
+EELAYER 25 0
 EELAYER END
 $Descr A4 11693 8268
@@
 AR Path="/556D3024/556D27D7" Ref="L3"  Part="1"
 AR Path="/556D375F/556D27D7" Ref="L4"  Part="1"
-F 0 "L2" V 7100 3300 40  0000 C CNN
+F 0 "L4" V 7100 3300 40  0000 C CNN
 F 1 "100u" V 7250 3300 40  0000 C CNN
-F 2 "~" H 7150 3300 60  0000 C CNN
+F 2 "custom:NRS6028T101MMGJ" H 7150 3300 60  0001 C CNN
 F 3 "~" H 7150 3300 60  0000 C CNN
 F 4 "MSS6132-823ML_" V 7150 3300 60  0001 C CNN "PartNumber"
@@
 AR Path="/556D3024/556D2801" Ref="D6"  Part="1"
 AR Path="/556D375F/556D2801" Ref="D7"  Part="1"
-F 0 "D5" H 6550 3100 40  0000 C CNN
+F 0 "D7" H 6550 3100 40  0000 C CNN
 F 1 "STPS1H100U" H 6550 2900 40  0000 C CNN
-F 2 "~" H 6550 3000 60  0000 C CNN
+F 2 "Diodes_SMD:SMB_Standard" H 6550 3000 60  0000 C CNN
 F 3 "~" H 6550 3000 60  0000 C CNN
 	1    6550 3000
@@
 Connection ~ 6550 3300
 $Comp
-L GND #PWR036
+L GND-RESCUE-led_spot #PWR45
 U 1 1 556D2B65
 P 6050 4150
-AR Path="/556D27B1/556D2B65" Ref="#PWR036"  Part="1"
-AR Path="/556D3024/556D2B65" Ref="#PWR045"  Part="1"
-AR Path="/556D375F/556D2B65" Ref="#PWR054"  Part="1"
-F 0 "#PWR036" H 6050 4150 30  0001 C CNN
+AR Path="/556D27B1/556D2B65" Ref="#PWR45"  Part="1"
+AR Path="/556D3024/556D2B65" Ref="#PWR55"  Part="1"
+AR Path="/556D375F/556D2B65" Ref="#PWR65"  Part="1"
+AR Path="/556D2B65" Ref="#PWR036"  Part="1"
+F 0 "#PWR65" H 6050 4150 30  0001 C CNN
 F 1 "GND" H 6050 4080 30  0001 C CNN
 F 2 "" H 6050 4150 60  0000 C CNN
@@
 $EndComp
 $Comp
-L R R8
+L R-RESCUE-led_spot R8
 U 1 1 556D2B74
 P 6050 3800
@@
 AR Path="/556D3024/556D2B74" Ref="R10"  Part="1"
 AR Path="/556D375F/556D2B74" Ref="R12"  Part="1"
-F 0 "R8" V 6130 3800 40  0000 C CNN
+AR Path="/556D2B74" Ref="R8"  Part="1"
+F 0 "R12" V 6130 3800 40  0000 C CNN
 F 1 "22K" V 6057 3801 40  0000 C CNN
-F 2 "~" V 5980 3800 30  0000 C CNN
+F 2 "Resistors_SMD:R_0603" V 5980 3800 30  0001 C CNN
 F 3 "~" H 6050 3800 30  0000 C CNN
 	1    6050 3800
@@
 Wire Wire Line
 	6050 3500 6050 3550
-Text HLabel 6150 3400 2    60   Input ~ 0
+Text HLabel 6350 3400 2    60   Input ~ 0
 DIM
 Wire Wire Line
-	6150 3400 5950 3400
-$Comp
-L GND #PWR037
+	5950 3400 6350 3400
+$Comp
+L GND-RESCUE-led_spot #PWR40
 U 1 1 556D2BA7
 P 4250 4150
-AR Path="/556D27B1/556D2BA7" Ref="#PWR037"  Part="1"
-AR Path="/556D3024/556D2BA7" Ref="#PWR046"  Part="1"
-AR Path="/556D375F/556D2BA7" Ref="#PWR055"  Part="1"
-F 0 "#PWR037" H 4250 4150 30  0001 C CNN
+AR Path="/556D27B1/556D2BA7" Ref="#PWR40"  Part="1"
+AR Path="/556D3024/556D2BA7" Ref="#PWR50"  Part="1"
+AR Path="/556D375F/556D2BA7" Ref="#PWR60"  Part="1"
+AR Path="/556D2BA7" Ref="#PWR037"  Part="1"
+F 0 "#PWR60" H 4250 4150 30  0001 C CNN
 F 1 "GND" H 4250 4080 30  0001 C CNN
 F 2 "" H 4250 4150 60  0000 C CNN
@@
 	4250 3500 4350 3500
 $Comp
-L R R7
+L R-RESCUE-led_spot R7
 U 1 1 556D2BC1
 P 4100 3800
@@
 AR Path="/556D3024/556D2BC1" Ref="R9"  Part="1"
 AR Path="/556D375F/556D2BC1" Ref="R11"  Part="1"
-F 0 "R7" V 4180 3800 40  0000 C CNN
+AR Path="/556D2BC1" Ref="R7"  Part="1"
+F 0 "R11" V 4180 3800 40  0000 C CNN
 F 1 "3K3" V 4107 3801 40  0000 C CNN
-F 2 "~" V 4030 3800 30  0000 C CNN
+F 2 "Resistors_SMD:R_0603" V 4030 3800 30  0001 C CNN
 F 3 "~" H 4100 3800 30  0000 C CNN
 	1    4100 3800
@@
 	4100 3400 4350 3400
 $Comp
-L GND #PWR038
+L GND-RESCUE-led_spot #PWR39
 U 1 1 556D2BD6
 P 4100 4150
-AR Path="/556D27B1/556D2BD6" Ref="#PWR038"  Part="1"
-AR Path="/556D3024/556D2BD6" Ref="#PWR047"  Part="1"
-AR Path="/556D375F/556D2BD6" Ref="#PWR056"  Part="1"
-F 0 "#PWR038" H 4100 4150 30  0001 C CNN
+AR Path="/556D27B1/556D2BD6" Ref="#PWR39"  Part="1"
+AR Path="/556D3024/556D2BD6" Ref="#PWR49"  Part="1"
+AR Path="/556D375F/556D2BD6" Ref="#PWR59"  Part="1"
+AR Path="/556D2BD6" Ref="#PWR038"  Part="1"
+F 0 "#PWR59" H 4100 4150 30  0001 C CNN
 F 1 "GND" H 4100 4080 30  0001 C CNN
 F 2 "" H 4100 4150 60  0000 C CNN
@@
 	4100 4150 4100 4050
 $Comp
-L GND #PWR039
+L GND-RESCUE-led_spot #PWR38
 U 1 1 556D2BEF
 P 3950 4150
-AR Path="/556D27B1/556D2BEF" Ref="#PWR039"  Part="1"
-AR Path="/556D3024/556D2BEF" Ref="#PWR048"  Part="1"
-AR Path="/556D375F/556D2BEF" Ref="#PWR057"  Part="1"
-F 0 "#PWR039" H 3950 4150 30  0001 C CNN
+AR Path="/556D27B1/556D2BEF" Ref="#PWR38"  Part="1"
+AR Path="/556D3024/556D2BEF" Ref="#PWR48"  Part="1"
+AR Path="/556D375F/556D2BEF" Ref="#PWR58"  Part="1"
+AR Path="/556D2BEF" Ref="#PWR039"  Part="1"
+F 0 "#PWR58" H 3950 4150 30  0001 C CNN
 F 1 "GND" H 3950 4080 30  0001 C CNN
 F 2 "" H 3950 4150 60  0000 C CNN
@@
 	3950 3300 4350 3300
 $Comp
-L C C5
+L C-RESCUE-led_spot C5
 U 1 1 556D2C12
 P 3800 3800
@@
 AR Path="/556D3024/556D2C12" Ref="C6"  Part="1"
 AR Path="/556D375F/556D2C12" Ref="C7"  Part="1"
-F 0 "C5" H 3800 3900 40  0000 L CNN
+AR Path="/556D2C12" Ref="C5"  Part="1"
+F 0 "C7" H 3800 3900 40  0000 L CNN
 F 1 "1u" H 3806 3715 40  0000 L CNN
-F 2 "~" H 3838 3650 30  0000 C CNN
+F 2 "Capacitors_SMD:C_0603" H 3838 3650 30  0000 C CNN
 F 3 "~" H 3800 3800 60  0000 C CNN
 	1    3800 3800
@@
 	3800 3200 4350 3200
 $Comp
-L GND #PWR040
+L GND-RESCUE-led_spot #PWR37
 U 1 1 556D2C35
 P 3800 4150
-AR Path="/556D27B1/556D2C35" Ref="#PWR040"  Part="1"
-AR Path="/556D3024/556D2C35" Ref="#PWR049"  Part="1"
-AR Path="/556D375F/556D2C35" Ref="#PWR058"  Part="1"
-F 0 "#PWR040" H 3800 4150 30  0001 C CNN
+AR Path="/556D27B1/556D2C35" Ref="#PWR37"  Part="1"
+AR Path="/556D3024/556D2C35" Ref="#PWR47"  Part="1"
+AR Path="/556D375F/556D2C35" Ref="#PWR57"  Part="1"
+AR Path="/556D2C35" Ref="#PWR040"  Part="1"
+F 0 "#PWR57" H 3800 4150 30  0001 C CNN
 F 1 "GND" H 3800 4080 30  0001 C CNN
 F 2 "" H 3800 4150 60  0000 C CNN
@@
 	3800 4150 3800 4000
 $Comp
-L C C10
+L C-RESCUE-led_spot C10
 U 1 1 55711043
 P 5600 2500
@@
 AR Path="/556D3024/55711043" Ref="C11"  Part="1"
 AR Path="/556D375F/55711043" Ref="C12"  Part="1"
-F 0 "C10" H 5600 2600 40  0000 L CNN
+AR Path="/55711043" Ref="C10"  Part="1"
+F 0 "C12" H 5600 2600 40  0000 L CNN
 F 1 "100n" H 5606 2415 40  0000 L CNN
-F 2 "" H 5638 2350 30  0000 C CNN
+F 2 "Capacitors_SMD:C_0805" H 5638 2350 30  0001 C CNN
 F 3 "" H 5600 2500 60  0000 C CNN
 	1    5600 2500
@@
 $EndComp
 $Comp
-L GND #PWR041
+L GND-RESCUE-led_spot #PWR43
 U 1 1 55711052
 P 5600 2700
-AR Path="/556D27B1/55711052" Ref="#PWR041"  Part="1"
-AR Path="/556D3024/55711052" Ref="#PWR050"  Part="1"
-AR Path="/556D375F/55711052" Ref="#PWR059"  Part="1"
-F 0 "#PWR041" H 5600 2700 30  0001 C CNN
+AR Path="/556D27B1/55711052" Ref="#PWR43"  Part="1"
+AR Path="/556D3024/55711052" Ref="#PWR53"  Part="1"
+AR Path="/556D375F/55711052" Ref="#PWR63"  Part="1"
+AR Path="/55711052" Ref="#PWR041"  Part="1"
+F 0 "#PWR63" H 5600 2700 30  0001 C CNN
 F 1 "GND" H 5600 2630 30  0001 C CNN
 F 2 "" H 5600 2700 60  0000 C CNN
@@
 $EndComp
 $Comp
-L +48V #PWR042
+L +48V #PWR42
 U 1 1 55711228
 P 5600 2300
-AR Path="/556D27B1/55711228" Ref="#PWR042"  Part="1"
-AR Path="/556D3024/55711228" Ref="#PWR051"  Part="1"
-AR Path="/556D375F/55711228" Ref="#PWR060"  Part="1"
-F 0 "#PWR042" H 5600 2430 20  0001 C CNN
+AR Path="/556D27B1/55711228" Ref="#PWR42"  Part="1"
+AR Path="/556D3024/55711228" Ref="#PWR52"  Part="1"
+AR Path="/556D375F/55711228" Ref="#PWR62"  Part="1"
+F 0 "#PWR62" H 5600 2430 20  0001 C CNN
 F 1 "+48V" H 5600 2400 30  0000 C CNN
 F 2 "" H 5600 2300 60  0000 C CNN
@@
 $EndComp
 $Comp
-L +48V #PWR043
+L +48V #PWR44
 U 1 1 5571157A
 P 5950 2800
-AR Path="/556D27B1/5571157A" Ref="#PWR043"  Part="1"
-AR Path="/556D3024/5571157A" Ref="#PWR052"  Part="1"
-AR Path="/556D375F/5571157A" Ref="#PWR061"  Part="1"
-F 0 "#PWR043" H 5950 2930 20  0001 C CNN
+AR Path="/556D27B1/5571157A" Ref="#PWR44"  Part="1"
+AR Path="/556D3024/5571157A" Ref="#PWR54"  Part="1"
+AR Path="/556D375F/5571157A" Ref="#PWR64"  Part="1"
+F 0 "#PWR64" H 5950 2930 20  0001 C CNN
 F 1 "+48V" H 5950 2900 30  0000 C CNN
 F 2 "" H 5950 2800 60  0000 C CNN
@@
 AR Path="/556D3024/5570FE55" Ref="U6"  Part="1"
 AR Path="/556D375F/5570FE55" Ref="U7"  Part="1"
-F 0 "U5" H 5150 3400 60  0000 C CNN
+F 0 "U7" H 5150 3400 60  0000 C CNN
 F 1 "TPS92511" H 5150 3250 60  0000 C CNN
-F 2 "" H 5150 3350 60  0000 C CNN
+F 2 "Housings_SOIC:SOIC-8-1EP_3.9x4.9mm_Pitch1.27mm" H 5150 3350 60  0001 C CNN
 F 3 "" H 5150 3350 60  0000 C CNN
 	1    5150 3350
@@
 $EndComp
 $Comp
-L GND #PWR044
+L GND-RESCUE-led_spot #PWR41
 U 1 1 55710122
 P 5150 4150
-AR Path="/556D27B1/55710122" Ref="#PWR044"  Part="1"
-AR Path="/556D3024/55710122" Ref="#PWR053"  Part="1"
-AR Path="/556D375F/55710122" Ref="#PWR062"  Part="1"
-F 0 "#PWR044" H 5150 4150 30  0001 C CNN
+AR Path="/556D27B1/55710122" Ref="#PWR41"  Part="1"
+AR Path="/556D3024/55710122" Ref="#PWR51"  Part="1"
+AR Path="/556D375F/55710122" Ref="#PWR61"  Part="1"
+AR Path="/55710122" Ref="#PWR044"  Part="1"
+F 0 "#PWR61" H 5150 4150 30  0001 C CNN
 F 1 "GND" H 5150 4080 30  0001 C CNN
 F 2 "" H 5150 4150 60  0000 C CNN
@@
 Text Notes 6800 3150 0    60   ~ 0
 NRS6028T101MMGJ
+$Comp
+L R R13
+U 1 1 5AAEF58F
+P 6250 3800
+AR Path="/556D27B1/5AAEF58F" Ref="R13"  Part="1"
+AR Path="/556D3024/5AAEF58F" Ref="R14"  Part="1"
+AR Path="/556D375F/5AAEF58F" Ref="R15"  Part="1"
+F 0 "R15" V 6330 3800 50  0000 C CNN
+F 1 "1K" V 6250 3800 50  0000 C CNN
+F 2 "Resistors_SMD:R_0603" V 6180 3800 50  0001 C CNN
+F 3 "" H 6250 3800 50  0001 C CNN
+	1    6250 3800
+	1    0    0    -1
+$EndComp
+Wire Wire Line
+	6250 3650 6250 3400
+Connection ~ 6250 3400
+Wire Wire Line
+	6250 3950 6250 4050
+$Comp
+L GND #PWR46
+U 1 1 5AAEF612
+P 6250 4050
+AR Path="/556D27B1/5AAEF612" Ref="#PWR46"  Part="1"
+AR Path="/556D3024/5AAEF612" Ref="#PWR56"  Part="1"
+AR Path="/556D375F/5AAEF612" Ref="#PWR66"  Part="1"
+F 0 "#PWR66" H 6250 3800 50  0001 C CNN
+F 1 "GND" H 6250 3900 50  0000 C CNN
+F 2 "" H 6250 4050 50  0001 C CNN
+F 3 "" H 6250 4050 50  0001 C CNN
+	1    6250 4050
+	1    0    0    -1
+$EndComp
 $EndSCHEMATC

Commit message: finish updating LED spot
Parts:
- D5: symbol DIODE -> D
Connections:
- net +48V: now also D5.1 (K); no longer D5.2 (K)
- net at L2.1, U5.7 (LX): now also D5.2 (A); no longer D5.1 (A)
Changed lines of the file:
@@
 AR Path="/556D3024/556D27D7" Ref="L3"  Part="1"
 AR Path="/556D375F/556D27D7" Ref="L4"  Part="1"
-F 0 "L4" V 7100 3300 40  0000 C CNN
+F 0 "L2" V 7100 3300 40  0000 C CNN
 F 1 "100u" V 7250 3300 40  0000 C CNN
 F 2 "custom:NRS6028T101MMGJ" H 7150 3300 60  0001 C CNN
@@
 $EndComp
 $Comp
-L DIODE D5
+L D D5
 U 1 1 556D2801
 P 6550 3000
@@
 AR Path="/556D3024/556D2801" Ref="D6"  Part="1"
 AR Path="/556D375F/556D2801" Ref="D7"  Part="1"
-F 0 "D7" H 6550 3100 40  0000 C CNN
+F 0 "D5" H 6550 3100 40  0000 C CNN
 F 1 "STPS1H100U" H 6550 2900 40  0000 C CNN
-F 2 "Diodes_SMD:SMB_Standard" H 6550 3000 60  0000 C CNN
+F 2 "Diodes_SMD:SMB_Standard" H 6250 3150 60  0000 C CNN
 F 3 "~" H 6550 3000 60  0000 C CNN
 	1    6550 3000
-	0    -1   -1   0
+	0    1    1    0
 $EndComp
 Text HLabel 7750 3300 2    60   Input ~ 0
@@
 Connection ~ 6300 2800
 Wire Wire Line
-	6550 3200 6550 3300
+	6550 3150 6550 3300
 Connection ~ 6550 3300
 $Comp
-L GND-RESCUE-led_spot #PWR45
+L GND-RESCUE-led_spot #PWR037
 U 1 1 556D2B65
 P 6050 4150
-AR Path="/556D27B1/556D2B65" Ref="#PWR45"  Part="1"
-AR Path="/556D3024/556D2B65" Ref="#PWR55"  Part="1"
-AR Path="/556D375F/556D2B65" Ref="#PWR65"  Part="1"
+AR Path="/556D27B1/556D2B65" Ref="#PWR037"  Part="1"
+AR Path="/556D3024/556D2B65" Ref="#PWR047"  Part="1"
+AR Path="/556D375F/556D2B65" Ref="#PWR057"  Part="1"
 AR Path="/556D2B65" Ref="#PWR036"  Part="1"
-F 0 "#PWR65" H 6050 4150 30  0001 C CNN
+F 0 "#PWR057" H 6050 4150 30  0001 C CNN
 F 1 "GND" H 6050 4080 30  0001 C CNN
 F 2 "" H 6050 4150 60  0000 C CNN
@@
 AR Path="/556D375F/556D2B74" Ref="R12"  Part="1"
 AR Path="/556D2B74" Ref="R8"  Part="1"
-F 0 "R12" V 6130 3800 40  0000 C CNN
+F 0 "R8" V 6130 3800 40  0000 C CNN
 F 1 "22K" V 6057 3801 40  0000 C CNN
 F 2 "Resistors_SMD:R_0603" V 5980 3800 30  0001 C CNN
@@
 	5950 3400 6350 3400
 $Comp
-L GND-RESCUE-led_spot #PWR40
+L GND-RESCUE-led_spot #PWR038
 U 1 1 556D2BA7
 P 4250 4150
-AR Path="/556D27B1/556D2BA7" Ref="#PWR40"  Part="1"
-AR Path="/556D3024/556D2BA7" Ref="#PWR50"  Part="1"
-AR Path="/556D375F/556D2BA7" Ref="#PWR60"  Part="1"
+AR Path="/556D27B1/556D2BA7" Ref="#PWR038"  Part="1"
+AR Path="/556D3024/556D2BA7" Ref="#PWR048"  Part="1"
+AR Path="/556D375F/556D2BA7" Ref="#PWR058"  Part="1"
 AR Path="/556D2BA7" Ref="#PWR037"  Part="1"
-F 0 "#PWR60" H 4250 4150 30  0001 C CNN
+F 0 "#PWR058" H 4250 4150 30  0001 C CNN
 F 1 "GND" H 4250 4080 30  0001 C CNN
 F 2 "" H 4250 4150 60  0000 C CNN
@@
 AR Path="/556D375F/556D2BC1" Ref="R11"  Part="1"
 AR Path="/556D2BC1" Ref="R7"  Part="1"
-F 0 "R11" V 4180 3800 40  0000 C CNN
+F 0 "R7" V 4180 3800 40  0000 C CNN
 F 1 "3K3" V 4107 3801 40  0000 C CNN
 F 2 "Resistors_SMD:R_0603" V 4030 3800 30  0001 C CNN
@@
 	4100 3400 4350 3400
 $Comp
-L GND-RESCUE-led_spot #PWR39
+L GND-RESCUE-led_spot #PWR039
 U 1 1 556D2BD6
 P 4100 4150
-AR Path="/556D27B1/556D2BD6" Ref="#PWR39"  Part="1"
-AR Path="/556D3024/556D2BD6" Ref="#PWR49"  Part="1"
-AR Path="/556D375F/556D2BD6" Ref="#PWR59"  Part="1"
+AR Path="/556D27B1/556D2BD6" Ref="#PWR039"  Part="1"
+AR Path="/556D3024/556D2BD6" Ref="#PWR049"  Part="1"
+AR Path="/556D375F/556D2BD6" Ref="#PWR059"  Part="1"
 AR Path="/556D2BD6" Ref="#PWR038"  Part="1"
-F 0 "#PWR59" H 4100 4150 30  0001 C CNN
+F 0 "#PWR059" H 4100 4150 30  0001 C CNN
 F 1 "GND" H 4100 4080 30  0001 C CNN
 F 2 "" H 4100 4150 60  0000 C CNN
@@
 	4100 4150 4100 4050
 $Comp
-L GND-RESCUE-led_spot #PWR38
+L GND-RESCUE-led_spot #PWR040
 U 1 1 556D2BEF
 P 3950 4150
-AR Path="/556D27B1/556D2BEF" Ref="#PWR38"  Part="1"
-AR Path="/556D3024/556D2BEF" Ref="#PWR48"  Part="1"
-AR Path="/556D375F/556D2BEF" Ref="#PWR58"  Part="1"
+AR Path="/556D27B1/556D2BEF" Ref="#PWR040"  Part="1"
+AR Path="/556D3024/556D2BEF" Ref="#PWR050"  Part="1"
+AR Path="/556D375F/556D2BEF" Ref="#PWR060"  Part="1"
 AR Path="/556D2BEF" Ref="#PWR039"  Part="1"
-F 0 "#PWR58" H 3950 4150 30  0001 C CNN
+F 0 "#PWR060" H 3950 4150 30  0001 C CNN
 F 1 "GND" H 3950 4080 30  0001 C CNN
 F 2 "" H 3950 4150 60  0000 C CNN
@@
 AR Path="/556D375F/556D2C12" Ref="C7"  Part="1"
 AR Path="/556D2C12" Ref="C5"  Part="1"
-F 0 "C7" H 3800 3900 40  0000 L CNN
+F 0 "C5" H 3800 3900 40  0000 L CNN
 F 1 "1u" H 3806 3715 40  0000 L CNN
 F 2 "Capacitors_SMD:C_0603" H 3838 3650 30  0000 C CNN
@@
 	3800 3200 4350 3200
 $Comp
-L GND-RESCUE-led_spot #PWR37
+L GND-RESCUE-led_spot #PWR041
 U 1 1 556D2C35
 P 3800 4150
-AR Path="/556D27B1/556D2C35" Ref="#PWR37"  Part="1"
-AR Path="/556D3024/556D2C35" Ref="#PWR47"  Part="1"
-AR Path="/556D375F/556D2C35" Ref="#PWR57"  Part="1"
+AR Path="/556D27B1/556D2C35" Ref="#PWR041"  Part="1"
+AR Path="/556D3024/556D2C35" Ref="#PWR051"  Part="1"
+AR Path="/556D375F/556D2C35" Ref="#PWR061"  Part="1"
 AR Path="/556D2C35" Ref="#PWR040"  Part="1"
-F 0 "#PWR57" H 3800 4150 30  0001 C CNN
+F 0 "#PWR061" H 3800 4150 30  0001 C CNN
 F 1 "GND" H 3800 4080 30  0001 C CNN
 F 2 "" H 3800 4150 60  0000 C CNN
@@
 AR Path="/556D375F/55711043" Ref="C12"  Part="1"
 AR Path="/55711043" Ref="C10"  Part="1"
-F 0 "C12" H 5600 2600 40  0000 L CNN
+F 0 "C10" H 5600 2600 40  0000 L CNN
 F 1 "100n" H 5606 2415 40  0000 L CNN
 F 2 "Capacitors_SMD:C_0805" H 5638 2350 30  0001 C CNN
@@
 $EndComp
 $Comp
-L GND-RESCUE-led_spot #PWR43
+L GND-RESCUE-led_spot #PWR042
 U 1 1 55711052
 P 5600 2700
-AR Path="/556D27B1/55711052" Ref="#PWR43"  Part="1"
-AR Path="/556D3024/55711052" Ref="#PWR53"  Part="1"
-AR Path="/556D375F/55711052" Ref="#PWR63"  Part="1"
+AR Path="/556D27B1/55711052" Ref="#PWR042"  Part="1"
+AR Path="/556D3024/55711052" Ref="#PWR052"  Part="1"
+AR Path="/556D375F/55711052" Ref="#PWR062"  Part="1"
 AR Path="/55711052" Ref="#PWR041"  Part="1"
-F 0 "#PWR63" H 5600 2700 30  0001 C CNN
+F 0 "#PWR062" H 5600 2700 30  0001 C CNN
 F 1 "GND" H 5600 2630 30  0001 C CNN
 F 2 "" H 5600 2700 60  0000 C CNN
@@
 $EndComp
 $Comp
-L +48V #PWR42
+L +48V #PWR043
 U 1 1 55711228
 P 5600 2300
-AR Path="/556D27B1/55711228" Ref="#PWR42"  Part="1"
-AR Path="/556D3024/55711228" Ref="#PWR52"  Part="1"
-AR Path="/556D375F/55711228" Ref="#PWR62"  Part="1"
-F 0 "#PWR62" H 5600 2430 20  0001 C CNN
+AR Path="/556D27B1/55711228" Ref="#PWR043"  Part="1"
+AR Path="/556D3024/55711228" Ref="#PWR053"  Part="1"
+AR Path="/556D375F/55711228" Ref="#PWR063"  Part="1"
+F 0 "#PWR063" H 5600 2430 20  0001 C CNN
 F 1 "+48V" H 5600 2400 30  0000 C CNN
 F 2 "" H 5600 2300 60  0000 C CNN
@@
 $EndComp
 $Comp
-L +48V #PWR44
+L +48V #PWR044
 U 1 1 5571157A
 P 5950 2800
-AR Path="/556D27B1/5571157A" Ref="#PWR44"  Part="1"
-AR Path="/556D3024/5571157A" Ref="#PWR54"  Part="1"
-AR Path="/556D375F/5571157A" Ref="#PWR64"  Part="1"
-F 0 "#PWR64" H 5950 2930 20  0001 C CNN
+AR Path="/556D27B1/5571157A" Ref="#PWR044"  Part="1"
+AR Path="/556D3024/5571157A" Ref="#PWR054"  Part="1"
+AR Path="/556D375F/5571157A" Ref="#PWR064"  Part="1"
+F 0 "#PWR064" H 5950 2930 20  0001 C CNN
 F 1 "+48V" H 5950 2900 30  0000 C CNN
 F 2 "" H 5950 2800 60  0000 C CNN
@@
 AR Path="/556D3024/5570FE55" Ref="U6"  Part="1"
 AR Path="/556D375F/5570FE55" Ref="U7"  Part="1"
-F 0 "U7" H 5150 3400 60  0000 C CNN
+F 0 "U5" H 5150 3400 60  0000 C CNN
 F 1 "TPS92511" H 5150 3250 60  0000 C CNN
 F 2 "Housings_SOIC:SOIC-8-1EP_3.9x4.9mm_Pitch1.27mm" H 5150 3350 60  0001 C CNN
@@
 $EndComp
 $Comp
-L GND-RESCUE-led_spot #PWR41
+L GND-RESCUE-led_spot #PWR045
 U 1 1 55710122
 P 5150 4150
-AR Path="/556D27B1/55710122" Ref="#PWR41"  Part="1"
-AR Path="/556D3024/55710122" Ref="#PWR51"  Part="1"
-AR Path="/556D375F/55710122" Ref="#PWR61"  Part="1"
+AR Path="/556D27B1/55710122" Ref="#PWR045"  Part="1"
+AR Path="/556D3024/55710122" Ref="#PWR055"  Part="1"
+AR Path="/556D375F/55710122" Ref="#PWR065"  Part="1"
 AR Path="/55710122" Ref="#PWR044"  Part="1"
-F 0 "#PWR61" H 5150 4150 30  0001 C CNN
+F 0 "#PWR065" H 5150 4150 30  0001 C CNN
 F 1 "GND" H 5150 4080 30  0001 C CNN
 F 2 "" H 5150 4150 60  0000 C CNN
@@
 AR Path="/556D3024/5AAEF58F" Ref="R14"  Part="1"
 AR Path="/556D375F/5AAEF58F" Ref="R15"  Part="1"
-F 0 "R15" V 6330 3800 50  0000 C CNN
+F 0 "R13" V 6330 3800 50  0000 C CNN
 F 1 "1K" V 6250 3800 50  0000 C CNN
 F 2 "Resistors_SMD:R_0603" V 6180 3800 50  0001 C CNN
@@
 	6250 3950 6250 4050
 $Comp
-L GND #PWR46
+L GND #PWR046
 U 1 1 5AAEF612
 P 6250 4050
-AR Path="/556D27B1/5AAEF612" Ref="#PWR46"  Part="1"
-AR Path="/556D3024/5AAEF612" Ref="#PWR56"  Part="1"
-AR Path="/556D375F/5AAEF612" Ref="#PWR66"  Part="1"
-F 0 "#PWR66" H 6250 3800 50  0001 C CNN
+AR Path="/556D27B1/5AAEF612" Ref="#PWR046"  Part="1"
+AR Path="/556D3024/5AAEF612" Ref="#PWR056"  Part="1"
+AR Path="/556D375F/5AAEF612" Ref="#PWR066"  Part="1"
+F 0 "#PWR066" H 6250 3800 50  0001 C CNN
 F 1 "GND" H 6250 3900 50  0000 C CNN
 F 2 "" H 6250 4050 50  0001 C CNN
@@
 	1    0    0    -1
 $EndComp
+Wire Wire Line
+	6550 2800 6550 2850
 $EndSCHEMATC
