File: led_spot_hardware/led spot.sch (KiCad schematic (older format))
At the start: 24 parts, among them K1 PWR, P1 mod_jack_in, P2 LED, P3 SWD, Q1 FDN5618P, U1 LM2594-HV, U2 STM32F030-20, U3 2CH-TVS, U4 ISL83485IBZ

Commit message: improvements to LED spot
Parts:
- added SW1: SW_Push, Buttons_Switches_SMD:SW_SPST_EVQPE1, symbol SW_Push
- C1, C9: footprint (none) -> Capacitors_SMD:C_0603; symbol C -> C-RESCUE-led_spot
- C2: footprint ~ -> Capacitors_SMD:C_0603; symbol C -> C-RESCUE-led_spot
- C3: footprint (none) -> Capacitors_SMD:C_0805; symbol C -> C-RESCUE-led_spot
- C8: footprint (none) -> Capacitors_SMD:C_1210; symbol C -> C-RESCUE-led_spot
- D1, D2: footprint (none) -> Diodes_SMD:SMB_Standard
- D4: footprint ~ -> LEDs:LED_0603; symbol LED -> LED-RESCUE-led_spot
- K1: footprint (none) -> Pin_Headers:Pin_Header_Straight_1x03
- L1: footprint (none) -> custom:VLF-M
- P1: footprint (none) -> custom:Assman-6p4c
- P2: footprint (none) -> custom:CHINESE-LARGE-LED
- P3: footprint (none) -> Pin_Headers:Pin_Header_Straight_1x04
- Q1, U3: footprint (none) -> TO_SOT_Packages_SMD:SOT-23
- R1, R2, R3, R4, R5: footprint (none) -> Resistors_SMD:R_0603; symbol R -> R-RESCUE-led_spot
- R6: footprint ~ -> Resistors_SMD:R_0603; symbol R -> R-RESCUE-led_spot
- U1, U4: footprint (none) -> Housings_SOIC:SOIC-8_3.9x4.9mm_Pitch1.27mm
- U2: footprint MODULE -> Housings_SSOP:TSSOP-20_4.4x6.5mm_Pitch0.65mm
Connections:
- net labels added: USR_BUTTON
- wire segments 73 -> 77
- no-connect marks 7 -> 6

Commit message: finish updating LED spot
Parts:
- D1, D2: symbol DIODESCH -> D_Schottky
- D4: symbol LED-RESCUE-led_spot -> LED
- Q1: symbol MOSFET_P -> Q_PMOS_GSD
Other:
- moved on the sheet: D1, D2, D4

Commit message: rev 2 gerbers
Other:
- note added: "VLS252012CX-220M-1"
- note removed: "VLF252012MT-220M"
Changed lines of the file:
@@
 $EndComp
 Text Notes 3350 950  0    60   ~ 0
-VLF252012MT-220M
+VLS252012CX-220M-1
 $Comp
 L VCC #PWR032
